Commit message: Update robot.xacro

File: robot_description/urdf/robot.xacro (robot description, xacro)
@@ -88,5 +88,5 @@
   <parent link="base_link"/>
   <child link="left_wheel_1"/>
-  <axis xyz="-0.0 1.0 0.0"/>
+  <axis xyz="0.0 1.0 0.0"/>
 </joint>
 <joint name="Rev2" type="continuous">
@@ -94,5 +94,5 @@
   <parent link="base_link"/>
   <child link="right_wheel_1"/>
-  <axis xyz="0.0 -1.0 -0.0"/>
+  <axis xyz="0.0 1.0 0.0"/>
 </joint>
 <joint name="Rigid3" type="fixed">
